File: Eagle/Whammy/whammy-schematic.sch (EAGLE design)
At the start: 0 parts

Commit message: Adding Eagle files.
Parts:
- added 3P3VREGULATOR: V_REG_LD1117VXX, SparkFun-IC-Power:V_REG_LD1117VXX
- added C1: 0.1uF, SparkFun-Capacitors:0.1UF-KIT-EZ-50V-20%
- added C2: 10uF, SparkFun-Capacitors:10UF-POLAR-RADIAL-2.5MM-25V-20%
- added J1: POWER_JACK, SparkFun-Connectors:POWER_JACK
- added LCD1: LCD-16X2SILK, SparkFun-Displays:LCD-16X2SILK
- added U$1: TEENSY_3.1-3.2_DIL, Teensy_3_and_LC_Series_Boards_v1.4:TEENSY_3.1-3.2_DIL
- added VR1: 10k, SparkFun-Resistors:TRIMPOT-PTH-10MM-KNOB-1/2W-10%
Connections:
- new net 3P3V: 3P3VREGULATOR.OUT, C2.+, LCD1.A, LCD1.E, LCD1.VDD, VR1.CCW
- new net DB4: LCD1.DB4
- new net DB5: LCD1.DB5
- new net DB6: LCD1.DB6
- new net DB7: LCD1.DB7
- new net GND: 3P3VREGULATOR.GND, C1.2, C2.-, J1.GND, J1.GNDBREAK, LCD1.K, LCD1.VSS, VR1.CW
- new net N$1: 3P3VREGULATOR.IN, C1.1, J1.PWR
- new net RS: LCD1.RS
- new net RW: LCD1.R/W
- new net VO: LCD1.VO, VR1.WIPER
