File: Eagle/Whammy/whammy-schematic.sch (EAGLE design)
At the start: 17 parts, among them J1 POWER_JACK, J2 DIN5, J3 UP, J4 DOWN, U1 5V REGULATOR

Commit message: Finished board with planes. Including OSHPark design rules file.
Parts:
- C1: device SparkFun-Capacitors:0.1UF-KIT-EZ-50V-20% -> SparkFun-Capacitors:22PF-PTH-2.54MM-200V-5%
- renumbered U$1 to U2
Changed lines of the file:
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@@
 </classes>
 <parts>
-<part name="U$1" library="Teensy_3_and_LC_Series_Boards_v1.4" deviceset="TEENSY_3.1-3.2_DIL" device=""/>
-<part name="C1" library="SparkFun-Capacitors" deviceset="0.1UF" device="-KIT-EZ-50V-20%" value="0.33uF"/>
+<part name="U2" library="Teensy_3_and_LC_Series_Boards_v1.4" deviceset="TEENSY_3.1-3.2_DIL" device=""/>
 <part name="C2" library="SparkFun-Capacitors" deviceset="10UF-POLAR" device="-RADIAL-2.5MM-25V-20%" value="0.1uF"/>
 <part name="GND2" library="SparkFun-PowerSymbols" deviceset="GND" device=""/>
@@
 <part name="H4" library="SparkFun-Hardware" deviceset="STAND-OFF" device=""/>
 <part name="J9" library="SparkFun-Connectors" deviceset="CONN_04" device=""/>
+<part name="C1" library="SparkFun-Capacitors" deviceset="22PF" device="-PTH-2.54MM-200V-5%" value="0.33uF"/>
 </parts>
 <sheets>
@@
 </plain>
 <instances>
-<instance part="U$1" gate="G$1" x="127" y="66.04"/>
-<instance part="C1" gate="G$1" x="0" y="124.46"/>
-<instance part="C2" gate="G$1" x="50.8" y="129.54"/>
+<instance part="U2" gate="G$1" x="127" y="66.04" smashed="yes">
+<attribute name="NAME" x="121.412" y="97.79" size="1.27" layer="95" font="vector" ratio="15"/>
+<attribute name="VALUE" x="119.888" y="25.146" size="1.27" layer="96" font="vector" ratio="15"/>
+</instance>
+<instance part="C2" gate="G$1" x="50.8" y="129.54" smashed="yes">
+<attribute name="NAME" x="51.816" y="130.175" size="1.778" layer="95" font="vector"/>
+<attribute name="VALUE" x="51.816" y="125.349" size="1.778" layer="96" font="vector"/>
+</instance>
 <instance part="GND2" gate="1" x="20.32" y="111.76"/>
-<instance part="J1" gate="G$1" x="-22.86" y="127"/>
-<instance part="LCD1" gate="G$1" x="2.54" y="81.28" rot="R180"/>
-<instance part="VR1" gate="R?" x="134.62" y="124.46"/>
+<instance part="J1" gate="G$1" x="-22.86" y="127" smashed="yes">
+<attribute name="VALUE" x="-33.02" y="137.16" size="1.778" layer="96" font="vector"/>
+<attribute name="NAME" x="-33.02" y="127" size="1.778" layer="95" font="vector"/>
+</instance>
+<instance part="LCD1" gate="G$1" x="2.54" y="81.28" smashed="yes" rot="R180">
+<attribute name="NAME" x="10.16" y="57.912" size="1.778" layer="95" rot="R180"/>
+<attribute name="VALUE" x="10.16" y="102.362" size="1.778" layer="96" rot="R180" align="top-left"/>
+</instance>
+<instance part="VR1" gate="R?" x="134.62" y="124.46" smashed="yes">
+<attribute name="NAME" x="133.096" y="127" size="1.778" layer="95" font="vector" rot="R90"/>
+<attribute name="VALUE" x="136.144" y="127" size="1.778" layer="96" font="vector" rot="R90" align="top-left"/>
+</instance>
 <instance part="GND1" gate="1" x="134.62" y="114.3"/>
-<instance part="J2" gate="G$1" x="33.02" y="22.86"/>
+<instance part="J2" gate="G$1" x="33.02" y="22.86" smashed="yes">
+<attribute name="NAME" x="33.02" y="17.272" size="1.778" layer="95" font="vector" align="bottom-center"/>
+<attribute name="VALUE" x="33.02" y="14.986" size="1.778" layer="96" font="vector" align="top-center"/>
+</instance>
 <instance part="R1" gate="G$1" x="12.7" y="27.94"/>
 <instance part="R2" gate="G$1" x="55.88" y="27.94"/>
-<instance part="J3" gate="G$1" x="33.02" y="-2.54"/>
-<instance part="J4" gate="G$1" x="33.02" y="-20.32"/>
-<instance part="U1" gate="G$1" x="20.32" y="134.62"/>
+<instance part="J3" gate="G$1" x="33.02" y="-2.54" smashed="yes">
+<attribute name="VALUE" x="30.48" y="-7.366" size="1.778" layer="96" font="vector"/>
+<attribute name="NAME" x="30.48" y="3.048" size="1.778" layer="95" font="vector"/>
+</instance>
+<instance part="J4" gate="G$1" x="33.02" y="-20.32" smashed="yes">
+<attribute name="VALUE" x="30.48" y="-25.146" size="1.778" layer="96" font="vector"/>
+<attribute name="NAME" x="30.48" y="-14.732" size="1.778" layer="95" font="vector"/>
+</instance>
+<instance part="U1" gate="G$1" x="20.32" y="134.62" smashed="yes">
+<attribute name="NAME" x="22.86" y="127" size="1.778" layer="95"/>
+<attribute name="VALUE" x="22.86" y="124.46" size="1.778" layer="96"/>
+</instance>
 <instance part="H1" gate="G$1" x="91.44" y="142.24"/>
 <instance part="H2" gate="G$1" x="96.52" y="142.24"/>
 <instance part="H3" gate="G$1" x="101.6" y="142.24"/>
 <instance part="H4" gate="G$1" x="106.68" y="142.24"/>
-<instance part="J9" gate="G$1" x="93.98" y="121.92"/>
+<instance part="J9" gate="G$1" x="93.98" y="121.92" smashed="yes">
+<attribute name="VALUE" x="88.9" y="114.554" size="1.778" layer="96" font="vector"/>
+<attribute name="NAME" x="88.9" y="130.048" size="1.778" layer="95" font="vector"/>
+</instance>
+<instance part="C1" gate="G$1" x="0" y="124.46" smashed="yes">
+<attribute name="NAME" x="1.524" y="127.381" size="1.778" layer="95" font="vector"/>
+<attribute name="VALUE" x="1.524" y="122.301" size="1.778" layer="96" font="vector"/>
+</instance>
 </instances>
 <busses>
@@
 <pinref part="J1" gate="G$1" pin="PWR"/>
 <wire x1="-20.32" y1="134.62" x2="0" y2="134.62" width="0.1524" layer="91"/>
-<pinref part="C1" gate="G$1" pin="1"/>
 <wire x1="0" y1="134.62" x2="12.7" y2="134.62" width="0.1524" layer="91"/>
 <wire x1="0" y1="129.54" x2="0" y2="134.62" width="0.1524" layer="91"/>
@@
 <label x="-15.24" y="134.62" size="1.778" layer="95"/>
 <pinref part="U1" gate="G$1" pin="IN"/>
+<pinref part="C1" gate="G$1" pin="1"/>
 </segment>
 <segment>
@@
 <wire x1="-12.7" y1="129.54" x2="-12.7" y2="114.3" width="0.1524" layer="91"/>
 <junction x="-12.7" y="129.54"/>
-<pinref part="C1" gate="G$1" pin="2"/>
 <wire x1="0" y1="121.92" x2="0" y2="114.3" width="0.1524" layer="91"/>
 <wire x1="0" y1="114.3" x2="-12.7" y2="114.3" width="0.1524" layer="91"/>
@@
 <wire x1="50.8" y1="114.3" x2="20.32" y2="114.3" width="0.1524" layer="91"/>
 <pinref part="U1" gate="G$1" pin="GND"/>
+<pinref part="C1" gate="G$1" pin="2"/>
 </segment>
 <segment>
@@
 </segment>
 <segment>
-<pinref part="U$1" gate="G$1" pin="GND"/>
+<pinref part="U2" gate="G$1" pin="GND"/>
 <wire x1="149.86" y1="83.82" x2="157.48" y2="83.82" width="0.1524" layer="91"/>
 <label x="152.4" y="83.82" size="1.778" layer="95"/>
 </segment>
 <segment>
-<pinref part="U$1" gate="G$1" pin="AGND"/>
+<pinref part="U2" gate="G$1" pin="AGND"/>
 <wire x1="149.86" y1="71.12" x2="157.48" y2="71.12" width="0.1524" layer="91"/>
 <label x="152.4" y="71.12" size="1.778" layer="95"/>
@@
 </segment>
 <segment>
-<pinref part="U$1" gate="G$1" pin="14/A1"/>
+<pinref part="U2" gate="G$1" pin="14/A1"/>
 <wire x1="104.14" y1="55.88" x2="88.9" y2="55.88" width="0.1524" layer="91"/>
 <label x="88.9" y="55.88" size="1.778" layer="95"/>
@@
 </segment>
 <segment>
-<pinref part="U$1" gate="G$1" pin="16/A2/T"/>
+<pinref part="U2" gate="G$1" pin="16/A2/T"/>
 <wire x1="104.14" y1="50.8" x2="88.9" y2="50.8" width="0.1524" layer="91"/>
 <label x="88.9" y="50.8" size="1.778" layer="95"/>
@@
 </segment>
 <segment>
-<pinref part="U$1" gate="G$1" pin="17/A3/T"/>
+<pinref part="U2" gate="G$1" pin="17/A3/T"/>
 <wire x1="104.14" y1="48.26" x2="88.9" y2="48.26" width="0.1524" layer="91"/>
 <label x="88.9" y="48.26" size="1.778" layer="95"/>
@@
 </segment>
 <segment>
-<pinref part="U$1" gate="G$1" pin="18/A4/T/SDA0"/>
+<pinref part="U2" gate="G$1" pin="18/A4/T/SDA0"/>
 <wire x1="104.14" y1="45.72" x2="88.9" y2="45.72" width="0.1524" layer="91"/>
 <label x="88.9" y="45.72" size="1.778" layer="95"/>
@@
 </segment>
 <segment>
-<pinref part="U$1" gate="G$1" pin="19/A5/T/SCL0"/>
+<pinref part="U2" gate="G$1" pin="19/A5/T/SCL0"/>
 <wire x1="104.14" y1="43.18" x2="88.9" y2="43.18" width="0.1524" layer="91"/>
 <label x="88.9" y="43.18" size="1.778" layer="95"/>
@@
 <net name="E" class="0">
 <segment>
-<pinref part="U$1" gate="G$1" pin="15/A1/T"/>
+<pinref part="U2" gate="G$1" pin="15/A1/T"/>
 <wire x1="104.14" y1="53.34" x2="88.9" y2="53.34" width="0.1524" layer="91"/>
 <label x="88.9" y="53.34" size="1.778" layer="95"/>
@@
 <net name="UP" class="0">
 <segment>
-<pinref part="U$1" gate="G$1" pin="2"/>
+<pinref part="U2" gate="G$1" pin="2"/>
 <wire x1="104.14" y1="86.36" x2="88.9" y2="86.36" width="0.1524" layer="91"/>
 <label x="88.9" y="86.36" size="1.778" layer="95"/>
@@
 <net name="DOWN" class="0">
 <segment>
-<pinref part="U$1" gate="G$1" pin="3/CAN-TX/PWM"/>
+<pinref part="U2" gate="G$1" pin="3/CAN-TX/PWM"/>
 <wire x1="104.14" y1="83.82" x2="88.9" y2="83.82" width="0.1524" layer="91"/>
 <label x="88.9" y="83.82" size="1.778" layer="95"/>
@@
 <net name="MIDIOUT" class="0">
 <segment>
-<pinref part="U$1" gate="G$1" pin="1/TX1/T"/>
+<pinref part="U2" gate="G$1" pin="1/TX1/T"/>
 <wire x1="104.14" y1="88.9" x2="88.9" y2="88.9" width="0.1524" layer="91"/>
 <label x="88.9" y="88.9" size="1.778" layer="95"/>
@@
 </segment>
 <segment>
-<pinref part="U$1" gate="G$1" pin="VIN"/>
+<pinref part="U2" gate="G$1" pin="VIN"/>
 <wire x1="149.86" y1="91.44" x2="157.48" y2="91.44" width="0.1524" layer="91"/>
 <label x="154.94" y="91.44" size="1.778" layer="95"/>
@@
 <net name="3P3V" class="0">
 <segment>
-<pinref part="U$1" gate="G$1" pin="3.3V"/>
+<pinref part="U2" gate="G$1" pin="3.3V"/>
 <wire x1="149.86" y1="88.9" x2="162.56" y2="88.9" width="0.1524" layer="91"/>
 <label x="152.4" y="88.9" size="1.778" layer="95"/>
